Commit message: threesixty camera code

File: cvg_sim_gazebo/urdf/quadrotor_sensors.urdf.xacro (robot description, xacro)
@@ -31,3 +31,7 @@
       <origin xyz="0.15 0.0 0.0" rpy="0 -${M_PI/2} 0"/>
     </xacro:generic_camera>
+    <include filename="$(find cvg_sim_gazebo)/urdf/sensors/360_camera.urdf.xacro" />
+    <xacro:threesixty_camera name="threesixty" sim_name="ardrone" parent="base_link" update_rate="60" res="640" image_format="R8G8B8">
+      <origin xyz="0.0 0.0 -0.15" rpy="0 0 0"/>
+    </xacro:threesixty_camera>
 </robot>
